File: USB_LEDs_2835_v3/USB_LEDs_2835_v3.kicad_sch (KiCad schematic)
At the start: 85 parts, among them J12 Screw_Terminal_01x03, J13 Barrel_Jack_Switch, U1 MT9284, U2 JL8022W-L, U3 74LVC1G04

Commit message: Add files via upload
Parts:
- removed D51, D52, D53, D54, D55, D56, D57, D58: 660nm, LED_SMD:LED_2835, symbol Device:LED_Small
- removed R102: 500k, Resistor_SMD:R_0402_1005Metric, symbol Device:R_Small_US
- added C6, C8: 22u, Capacitor_SMD:C_0603_1608Metric, symbol Device:C
- added C7: 200n, Capacitor_SMD:C_0603_1608Metric, symbol Device:C
- added C9: 100u/16V, Capacitor_Tantalum_SMD:CP_EIA-3528-21_Kemet-B, symbol Device:C_Polarized
- added J1: external header, Connector_PinHeader_2.54mm:PinHeader_1x05_P2.54mm_Vertical, symbol Connector:Conn_01x05_Male
- added J2: Fan conn, Connector:FanPinHeader_1x04_P2.54mm_Vertical_custom, symbol Connector:Conn_01x04_Male
- added JP1: j_open, TestPoint:TestPoint_2Pads_Pitch2.54mm_Drill0.8mm, symbol Jumper:Jumper_2_Open
- added L2: 4.7u, Inductor_SMD:L_0530_custom, symbol Device:L
- added R5: 51k, Resistor_SMD:R_0603_1608Metric, symbol Device:R_Small_US
- added R7: 6.8k, Resistor_SMD:R_0603_1608Metric, symbol Device:R_Small_US
- added R8: 22k, Resistor_SMD:R_0603_1608Metric, symbol Device:R_Small_US
- added U4: STI3470, Package_TO_SOT_SMD:SOT-23-6, symbol Regulator_Controller:STI3470
- C2, Cx1: value 1u -> 22u
- TP1: footprint TestPoint:TestPoint_Loop_D2.50mm_Drill1.0mm -> (none)
- renumbered D41 to D10, D45 to D11, D49 to D12, D9 to D13, D10 to D14, D11 to D15, D12 to D16, D13 to D17, D14 to D18, D15 to D19, D16 to D20, D38 to D21, D42 to D22, D46 to D23, D50 to D24, D17 to D25, D18 to D26, D19 to D27, D20 to D28, D21 to D29, D22 to D30, D23 to D31, D24 to D32, D36 to D33, D40 to D34, D44 to D35, D48 to D36, D25 to D37, D26 to D38, D27 to D39, D28 to D40, D29 to D41, D30 to D42, D31 to D43, D32 to D44, D35 to D45, D39 to D46, D43 to D47, D47 to D48, D33 to D49, D34 to D50, D37 to D9
Connections:
- net +12V: now also C6.1, C9.1, J1.2 (Pin_2), J2.2 (Pin_2), R8.2, U4.5 (IN)
- net +5V: now also J1.5 (Pin_5), JP1.2 (B)
- net GND: now also C6.2, C8.2, C9.2, J1.1 (Pin_1), J2.1 (Pin_1), R7.1, U4.2 (GND)
- net at Cx1.1, D1.2 (A), D13.2 (A)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: now also U1.5 (OV)
- net at R1.1, Rx1.2: now also D12.1 (K), D24.1 (K), D36.1 (K), D48.1 (K)
- net at D3.1 (K), D4.2 (A): no longer U1.5 (OV)
- new net: C7.1, U4.1 (BS)
- new net: C7.2, L2.1, U4.6 (LX)
- new net: J1.3 (Pin_3), J2.3 (Pin_3)
- new net: J1.4 (Pin_4), J2.4 (Pin_4)
- new net: R8.1, U4.4 (EN)
- new net: C8.1, JP1.1 (A), L2.2, R5.1
- new net: R5.2, R7.2, U4.3 (FB)

Commit message: Add files via upload
Parts:
- R2, R3: footprint Resistor_SMD:R_0402_1005Metric -> Resistor_SMD:R_0603_1608Metric
Changed lines of the file:
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@@
       (effects (font (size 1.27 1.27)) (justify left))
     )
-    (property "Footprint" "Resistor_SMD:R_0402_1005Metric" (id 2) (at 126.365 51.562 0)
+    (property "Footprint" "Resistor_SMD:R_0603_1608Metric" (id 2) (at 126.365 51.562 0)
       (effects (font (size 1.27 1.27)) hide)
     )
@@
       (effects (font (size 1.27 1.27)) (justify left))
     )
-    (property "Footprint" "Resistor_SMD:R_0402_1005Metric" (id 2) (at 121.285 43.942 0)
+    (property "Footprint" "Resistor_SMD:R_0603_1608Metric" (id 2) (at 121.285 43.942 0)
       (effects (font (size 1.27 1.27)) hide)
     )
@@
     )
     (path "/66fae963-db90-4b44-b511-1ffbefe55119"
-      (reference "R2") (unit 1) (value "10k") (footprint "Resistor_SMD:R_0402_1005Metric")
+      (reference "R2") (unit 1) (value "10k") (footprint "Resistor_SMD:R_0603_1608Metric")
     )
     (path "/2b40a6ef-b747-4e09-b1c9-aaa6bec91ed5"
-      (reference "R3") (unit 1) (value "10k") (footprint "Resistor_SMD:R_0402_1005Metric")
+      (reference "R3") (unit 1) (value "10k") (footprint "Resistor_SMD:R_0603_1608Metric")
     )
     (path "/b29813e7-e4cd-496d-bb16-c537eb2ab1d5"
